File: hardware/xiao-solar/xiao-solar.kicad_sch (KiCad schematic)
At the start: 81 parts, among them J1 SOLAR, J2 VIN2 5-20V, J3 NTC 10k (103AT), J4 BATTERY, J5 I2C rail, J6 LOAD_IN до 12V, J7 OUT1 heater, J8 OUT2 fan, J9 OUT3 spare, Q1 AO3400A, Q2 AO3400A (ship FET), Q3 FS8205A, Q4 AO3400A, Q5 AO3400A, Q6 AO3400A, U1 BQ25798RQMR, U2 DW01A, U3 XIAO nRF52840, U4 Wio-SX1262 for XIAO, U5 SHT40-AD1B, U6 PCA9685PW

Commit message: hardware/xiao-solar: LOAD_IN reverse-polarity P-FET, PCB placement v0.1
Review answers: Wio uses the XIAO footprint, I2C header SCL/SDA/3V3/GND,
3 outputs, ~3 A battery limit is enough (heater and fan never together).
tools/gen_pcb.py builds the board (48x86 mm, 2 layers, parts on top,
GND pour both sides); routing still to do.

Co-Authored-By: Claude Opus 5.5 <noreply@anthropic.com>
Claude-Session: https://claude.ai/code/session_01P5Km81NY9NPL6RpKFGVEbH
Parts:
- added Q7: AO3401A, Package_TO_SOT_SMD:SOT-23, symbol Device:Q_PMOS_GSD
- added R19: 22k, Resistor_SMD:R_0603_1608Metric, symbol Device:R
- added R20: 10k, Resistor_SMD:R_0603_1608Metric, symbol Device:R
Connections:
- net GND: now also R20.2
- net LOAD_IN: now also Q7.2 (S), R19.1; no longer J6.1 (Pin_1)
- new net LOAD_G: Q7.1 (G), R19.2, R20.1
- new net LOAD_IN_RAW: J6.1 (Pin_1), Q7.3 (D)
Changed lines of the file:
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@@
     (instances (project "xiao-solar" (path "/6b1f3c1e-6a5e-4b7e-9d65-5f0b3a1d0001" (reference "J6") (unit 1))))
+  )
+  (symbol (lib_id "Device:Q_PMOS_GSD") (at 270 195 0) (unit 1) (in_bom yes) (on_board yes) (dnp no)
+    (property "Reference" "Q7" (at 270 185.42 0) (effects (font (size 1.27 1.27))))
+    (property "Value" "AO3401A" (at 270 187.72 0) (effects (font (size 1.27 1.27))))
+    (property "Footprint" "Package_TO_SOT_SMD:SOT-23" (at 270 195 0) (effects (font (size 1.27 1.27)) hide))
+    (property "Datasheet" "" (at 270 195 0) (effects (font (size 1.27 1.27)) hide))
+    (property "LCSC" "C15127" (at 270 195 0) (effects (font (size 1.27 1.27)) hide))
+    (pin "1")
+    (pin "2")
+    (pin "3")
+    (instances (project "xiao-solar" (path "/6b1f3c1e-6a5e-4b7e-9d65-5f0b3a1d0001" (reference "Q7") (unit 1))))
+  )
+  (symbol (lib_id "Device:R") (at 262 205 0) (unit 1) (in_bom yes) (on_board yes) (dnp no)
+    (property "Reference" "R19" (at 264 204 0) (effects (font (size 1.27 1.27)) (justify left)))
+    (property "Value" "22k" (at 264 206.5 0) (effects (font (size 1.27 1.27)) (justify left)))
+    (property "Footprint" "Resistor_SMD:R_0603_1608Metric" (at 262 205 0) (effects (font (size 1.27 1.27)) hide))
+    (property "Datasheet" "" (at 262 205 0) (effects (font (size 1.27 1.27)) hide))
+    (property "LCSC" "C31850" (at 262 205 0) (effects (font (size 1.27 1.27)) hide))
+    (pin "1")
+    (pin "2")
+    (instances (project "xiao-solar" (path "/6b1f3c1e-6a5e-4b7e-9d65-5f0b3a1d0001" (reference "R19") (unit 1))))
+  )
+  (symbol (lib_id "Device:R") (at 275 207 0) (unit 1) (in_bom yes) (on_board yes) (dnp no)
+    (property "Reference" "R20" (at 277 206 0) (effects (font (size 1.27 1.27)) (justify left)))
+    (property "Value" "10k" (at 277 208.5 0) (effects (font (size 1.27 1.27)) (justify left)))
+    (property "Footprint" "Resistor_SMD:R_0603_1608Metric" (at 275 207 0) (effects (font (size 1.27 1.27)) hide))
+    (property "Datasheet" "" (at 275 207 0) (effects (font (size 1.27 1.27)) hide))
+    (property "LCSC" "C25804" (at 275 207 0) (effects (font (size 1.27 1.27)) hide))
+    (pin "1")
+    (pin "2")
+    (instances (project "xiao-solar" (path "/6b1f3c1e-6a5e-4b7e-9d65-5f0b3a1d0001" (reference "R20") (unit 1))))
   )
   (symbol (lib_id "Device:C") (at 300 172 0) (unit 1) (in_bom yes) (on_board yes) (dnp no)
@@
   (label "VLOAD" (at 285 175.81 270) (fields_autoplaced) (effects (font (size 1.0 1.0)) (justify right bottom)))
   (label "LOAD_IN" (at 290.08 172 0) (fields_autoplaced) (effects (font (size 1.0 1.0)) (justify left bottom)))
-  (label "LOAD_IN" (at 259.92 180 180) (fields_autoplaced) (effects (font (size 1.0 1.0)) (justify right bottom)))
+  (label "LOAD_IN_RAW" (at 259.92 180 180) (fields_autoplaced) (effects (font (size 1.0 1.0)) (justify right bottom)))
   (label "GND" (at 259.92 182.54 180) (fields_autoplaced) (effects (font (size 1.0 1.0)) (justify right bottom)))
+  (label "LOAD_G" (at 264.92 195 180) (fields_autoplaced) (effects (font (size 1.0 1.0)) (justify right bottom)))
+  (label "LOAD_IN" (at 272.54 200.08 270) (fields_autoplaced) (effects (font (size 1.0 1.0)) (justify right bottom)))
+  (label "LOAD_IN_RAW" (at 272.54 189.92 90) (fields_autoplaced) (effects (font (size 1.0 1.0)) (justify left bottom)))
+  (label "LOAD_IN" (at 262 201.19 90) (fields_autoplaced) (effects (font (size 1.0 1.0)) (justify left bottom)))
+  (label "LOAD_G" (at 262 208.81 270) (fields_autoplaced) (effects (font (size 1.0 1.0)) (justify right bottom)))
+  (label "LOAD_G" (at 275 203.19 90) (fields_autoplaced) (effects (font (size 1.0 1.0)) (justify left bottom)))
+  (label "GND" (at 275 210.81 270) (fields_autoplaced) (effects (font (size 1.0 1.0)) (justify right bottom)))
   (label "VLOAD" (at 300 168.19 90) (fields_autoplaced) (effects (font (size 1.0 1.0)) (justify left bottom)))
   (label "GND" (at 300 175.81 270) (fields_autoplaced) (effects (font (size 1.0 1.0)) (justify right bottom)))

Commit message: xiao-solar v0.2 WIP: Argon review fixes, layout and first routing
- CE straight on D0, JP2 selects pull-down (Li-ion, charges without the Xiao) or
  pull-up (LiFePO4, charges only after firmware set VREG); Q1/R5 removed
- VBUS/PMID caps 10uF/50V 1206; SMBJ24A and HJ8205 swapped to preferred parts
- charger laid out per the BQ25798 layout guide, TS divider and side-pin parts at U1,
  GND pin 27 runs under the package to pins 10/11 and a via
- SHT40 on a slotted tongue without copper pour
- LOAD_IN removed; loads on SYS through an LC filter (2.2uH + 2x22uF), PGND with a
  net tie, 1k gate resistors and 100nF across each output against radio noise
- four 2.8 mm mounting holes with 6 mm keepout, board 48x94 mm
- tools/route.py (Freerouting + SES import + GND stitching), refill.py, finish.py,
  export.py (Gerber/drill zip, JLC CPL); __pycache__ removed, .gitignore added
- 3 connections still unrouted (QON, BTST2, PWM1)

Co-Authored-By: Claude Opus 5.5 <noreply@anthropic.com>
Claude-Session: https://claude.ai/code/session_01P5Km81NY9NPL6RpKFGVEbH
Parts:
- removed J6: LOAD_IN до 12V, Connector_PinHeader_2.54mm:PinHeader_1x02_P2.54mm_Vertical, symbol Connector_Generic:Conn_01x02
- removed JP1: VLOAD: 1-2 SYS / 2-3 LOAD_IN, Jumper:SolderJumper-3_P1.3mm_Bridged12_RoundedPad1.0x1.5mm, symbol Jumper:SolderJumper_3_Bridged12
- removed Q1: AO3400A, Package_TO_SOT_SMD:SOT-23, symbol Transistor_FET:BSS138
- removed Q7: AO3401A, Package_TO_SOT_SMD:SOT-23, symbol Device:Q_PMOS_GSD
- removed R19: 22k, Resistor_SMD:R_0603_1608Metric, symbol Device:R
- removed R20: 10k, Resistor_SMD:R_0603_1608Metric, symbol Device:R
- removed R5: 100k, Resistor_SMD:R_0603_1608Metric, symbol Device:R
- added C26: 22u/25V, Capacitor_SMD:C_1206_3216Metric, symbol Device:C
- added C27, C28, C29, C30: 100n, Capacitor_SMD:C_0603_1608Metric, symbol Device:C
- added FB1: 2.2uH 3.2A, xiao_solar:IND-SMD_L4.0-W4.0_FNR40XXS, symbol xiao_solar:FNR4030S2R2MT
- added H3, H4: M2/M2.5, xiao_solar:MountingHole_2.8mm_Keepout6mm, symbol Mechanical:MountingHole
- added JP2: CE: 1-2 Li-ion / 2-3 LiFePO4, Jumper:SolderJumper-3_P1.3mm_Bridged12_RoundedPad1.0x1.5mm, symbol Jumper:SolderJumper_3_Bridged12
- added NT1: PGND-GND, NetTie:NetTie-2_SMD_Pad0.5mm, symbol Device:NetTie_2
- C1, C2, C6, C7, C8: value 10u/25V -> 10u/50V; footprint Capacitor_SMD:C_0805_2012Metric -> Capacitor_SMD:C_1206_3216Metric; LCSC C15850 -> C13585
- C25: value 10u/25V -> 22u/25V; footprint Capacitor_SMD:C_0805_2012Metric -> Capacitor_SMD:C_1206_3216Metric; LCSC C15850 -> C12891
- D3: LCSC C87268 -> C19077578
- H1, H2: value M2.5 -> M2/M2.5; footprint MountingHole:MountingHole_2.7mm_M2.5 -> xiao_solar:MountingHole_2.8mm_Keepout6mm
- Q3: value FS8205A -> HJ8205; LCSC C2830320 -> C20069150
- R13, R15, R17: value 100 -> 1k; LCSC C22775 -> C21190
Connections:
- net CHG_EN is gone; now on net CE: U3.1 (D0/A0)
- net 3V3: now also JP2.3 (B)
- net GND: now also JP2.1 (A), NT1.2; no longer C25.2, Q4.2 (S), Q5.2 (S), Q6.2 (S), R14.2, R16.2, R18.2
- net OUT1+: now also C28.1
- net OUT1-: now also C28.2
- net OUT2+: now also C29.1
- net OUT2-: now also C29.2
- net OUT3+: now also C30.1
- net OUT3-: now also C30.2
- net REGN: no longer R4.1
- net SYS: now also FB1.1
- net VLOAD: now also C26.1, C27.1, FB1.2
- new net CE_PULL: JP2.2 (C), R4.1
- new net PGND: C25.2, C26.2, C27.2, NT1.1, Q4.2 (S), Q5.2 (S), Q6.2 (S), R14.2, R16.2, R18.2
Other:
- note added: "3. БАТЕРИЯ 1S (Li-ion по подразбиране, LiFePO4 с настройка): ship FET + DW01A/HJ8205"
- note added: "CE: JP2 1-2 (Li-ion) зарежда и без Xiao; 2-3 (LiFePO4) само след запис на VREG и D0=0. Watchdog off. D+/D- не се ползват."
- note added: "събужда се само когато се появи напрежение от панела. DW01A: 2.4 V / 4.3 V резерв, HJ8205 в минуса."
- note removed: "3. БАТЕРИЯ 1S (Li-ion по подразбиране, LiFePO4 с настройка): ship FET + DW01A/FS8205A"
- note removed: "CE: R4 държи зареждането спряно; фърмуерът пуска D0 (CHG_EN) едва след запис на VREG. Watchdog off. D+/D- не се ползват."
- note removed: "събужда се само когато се появи напрежение от панела. DW01A: 2.4 V / 4.3 V резерв, FS8205A в минуса."

Commit message: xiao-solar v0.2: final routing, Gerber, JLC BOM/CPL
CE jumper JP2 (Li-ion/LiFePO4), INT left open, 4 mounting holes 2.8 mm
with 6 mm keep-out, LOAD_IN removed, load noise filtering (LC on VLOAD,
PGND star via net tie, 1k gates, 100n per output), fewer JLC extended
parts. Routing tools: finish.py second pass, patch_route.py grid A*.
DRC: 0 unconnected, only net-tie polygon clearance and cosmetic items.

Co-Authored-By: Claude Opus 5.5 <noreply@anthropic.com>
Claude-Session: https://claude.ai/code/session_01P5Km81NY9NPL6RpKFGVEbH
Parts:
- removed R7: 10k, Resistor_SMD:R_0603_1608Metric, symbol Device:R
- removed TP1: INT, TestPoint:TestPoint_Pad_D1.0mm, symbol Connector:TestPoint
Connections:
- net PWM1: now also U6.8 (LED2); no longer U6.6 (LED0)
- net PWM3: now also U6.6 (LED0); no longer U6.8 (LED2)
- net INT: no longer names the net of U1.21 (~{INT})
- no-connect marks 20 -> 21
Changed lines of the file:
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@@
     (instances (project "xiao-solar" (path "/6b1f3c1e-6a5e-4b7e-9d65-5f0b3a1d0001" (reference "D4") (unit 1))))
-  )
-  (symbol (lib_id "Device:R") (at 70 160 0) (unit 1) (in_bom yes) (on_board yes) (dnp no)
-    (property "Reference" "R7" (at 72 159 0) (effects (font (size 1.27 1.27)) (justify left)))
-    (property "Value" "10k" (at 72 161.5 0) (effects (font (size 1.27 1.27)) (justify left)))
-    (property "Footprint" "Resistor_SMD:R_0603_1608Metric" (at 70 160 0) (effects (font (size 1.27 1.27)) hide))
-    (property "Datasheet" "" (at 70 160 0) (effects (font (size 1.27 1.27)) hide))
-    (property "LCSC" "C25804" (at 70 160 0) (effects (font (size 1.27 1.27)) hide))
-    (pin "1")
-    (pin "2")
-    (instances (project "xiao-solar" (path "/6b1f3c1e-6a5e-4b7e-9d65-5f0b3a1d0001" (reference "R7") (unit 1))))
-  )
-  (symbol (lib_id "Connector:TestPoint") (at 80 165 0) (unit 1) (in_bom yes) (on_board yes) (dnp no)
-    (property "Reference" "TP1" (at 82 164 0) (effects (font (size 1.27 1.27)) (justify left)))
-    (property "Value" "INT" (at 82 166.5 0) (effects (font (size 1.27 1.27)) (justify left)))
-    (property "Footprint" "TestPoint:TestPoint_Pad_D1.0mm" (at 80 165 0) (effects (font (size 1.27 1.27)) hide))
-    (property "Datasheet" "" (at 80 165 0) (effects (font (size 1.27 1.27)) hide))
-    (property "LCSC" "" (at 80 165 0) (effects (font (size 1.27 1.27)) hide))
-    (pin "1")
-    (instances (project "xiao-solar" (path "/6b1f3c1e-6a5e-4b7e-9d65-5f0b3a1d0001" (reference "TP1") (unit 1))))
   )
   (symbol (lib_id "Connector:TestPoint") (at 90 165 0) (unit 1) (in_bom yes) (on_board yes) (dnp no)
@@
   (label "BTST2" (at 86.51 132.62 0) (fields_autoplaced) (effects (font (size 1.0 1.0)) (justify left bottom)))
   (label "PROG" (at 86.51 130.08 0) (fields_autoplaced) (effects (font (size 1.0 1.0)) (justify left bottom)))
-  (label "INT" (at 86.51 127.54 0) (fields_autoplaced) (effects (font (size 1.0 1.0)) (justify left bottom)))
   (label "BAT" (at 86.51 125 0) (fields_autoplaced) (effects (font (size 1.0 1.0)) (justify left bottom)))
   (label "BAT" (at 86.51 122.46 0) (fields_autoplaced) (effects (font (size 1.0 1.0)) (justify left bottom)))
@@
   (label "STAT" (at 51.19 175 180) (fields_autoplaced) (effects (font (size 1.0 1.0)) (justify right bottom)))
   (label "LED_STAT" (at 58.81 175 0) (fields_autoplaced) (effects (font (size 1.0 1.0)) (justify left bottom)))
-  (label "3V3" (at 70 156.19 90) (fields_autoplaced) (effects (font (size 1.0 1.0)) (justify left bottom)))
-  (label "INT" (at 70 163.81 270) (fields_autoplaced) (effects (font (size 1.0 1.0)) (justify right bottom)))
-  (label "INT" (at 80 165 270) (fields_autoplaced) (effects (font (size 1.0 1.0)) (justify right bottom)))
   (label "QON" (at 90 165 270) (fields_autoplaced) (effects (font (size 1.0 1.0)) (justify right bottom)))
   (label "BATT+" (at 14.92 230 180) (fields_autoplaced) (effects (font (size 1.0 1.0)) (justify right bottom)))
@@
   (label "GND" (at 227.3 206.11 180) (fields_autoplaced) (effects (font (size 1.0 1.0)) (justify right bottom)))
   (label "GND" (at 227.3 208.65 180) (fields_autoplaced) (effects (font (size 1.0 1.0)) (justify right bottom)))
-  (label "PWM1" (at 227.3 211.19 180) (fields_autoplaced) (effects (font (size 1.0 1.0)) (justify right bottom)))
+  (label "PWM3" (at 227.3 211.19 180) (fields_autoplaced) (effects (font (size 1.0 1.0)) (justify right bottom)))
   (label "PWM2" (at 227.3 213.73 180) (fields_autoplaced) (effects (font (size 1.0 1.0)) (justify right bottom)))
-  (label "PWM3" (at 227.3 216.27 180) (fields_autoplaced) (effects (font (size 1.0 1.0)) (justify right bottom)))
+  (label "PWM1" (at 227.3 216.27 180) (fields_autoplaced) (effects (font (size 1.0 1.0)) (justify right bottom)))
   (label "GND" (at 227.3 231.51 180) (fields_autoplaced) (effects (font (size 1.0 1.0)) (justify right bottom)))
   (label "GND" (at 252.7 211.19 0) (fields_autoplaced) (effects (font (size 1.0 1.0)) (justify left bottom)))
@@
   (no_connect (at 53.49 122.46))
   (no_connect (at 53.49 125))
+  (no_connect (at 86.51 127.54))
   (no_connect (at 140.16 252.54))
   (no_connect (at 286.03 37.38))

Commit message: hardware: xiao-solar v0.4 (no loads, INA219, 48x71.5) + block schematics for both boards
Co-Authored-By: Claude Opus 5.5 <noreply@anthropic.com>
Claude-Session: https://claude.ai/code/session_01P5Km81NY9NPL6RpKFGVEbH
Parts:
- removed C25, C26: 22u/25V, Capacitor_SMD:C_1206_3216Metric, symbol Device:C
- removed C27, C28, C29, C30: 100n, Capacitor_SMD:C_0603_1608Metric, symbol Device:C
- removed D5, D6, D7, D8: B5819W, Diode_SMD:D_SOD-123, symbol Device:D_Schottky
- removed F1, F2, F3: 2A/16V, Fuse:Fuse_1206_3216Metric, symbol Device:Polyfuse
- removed FB1: 2.2uH 3.2A, xiao_solar:IND-SMD_L4.0-W4.0_FNR40XXS, symbol xiao_solar:FNR4030S2R2MT
- removed J7: OUT1 heater, Connector_PinHeader_2.54mm:PinHeader_1x02_P2.54mm_Vertical, symbol Connector_Generic:Conn_01x02
- removed J8: OUT2 fan, Connector_PinHeader_2.54mm:PinHeader_1x02_P2.54mm_Vertical, symbol Connector_Generic:Conn_01x02
- removed J9: OUT3 spare, Connector_PinHeader_2.54mm:PinHeader_1x02_P2.54mm_Vertical, symbol Connector_Generic:Conn_01x02
- removed NT1: PGND-GND, NetTie:NetTie-2_SMD_Pad0.5mm, symbol Device:NetTie_2
- removed Q4, Q5, Q6: AO3400A, Package_TO_SOT_SMD:SOT-23, symbol Transistor_FET:BSS138
- removed R13, R15, R17: 1k, Resistor_SMD:R_0603_1608Metric, symbol Device:R
- removed R14, R16, R18: 100k, Resistor_SMD:R_0603_1608Metric, symbol Device:R
- removed U6: PCA9685PW, xiao_solar:TSSOP-28_L9.7-W4.4-P0.65-LS6.4-TL, symbol xiao_solar:PCA9685PW,118
- added D5: LM66100, Package_TO_SOT_SMD:SOT-363_SC-70-6, symbol xiao_solar:LM66100
- added JP3: no ship FET (LiFePO4), Jumper:SolderJumper-2_P1.3mm_Open_RoundedPad1.0x1.5mm, symbol Jumper:SolderJumper_2_Open
- added RS1: 0.05 1W, Resistor_SMD:R_1206_3216Metric, symbol Device:R
- added TP10: SDA, TestPoint:TestPoint_Pad_D1.0mm, symbol Connector:TestPoint
- added TP11: BATS, TestPoint:TestPoint_Pad_D1.0mm, symbol Connector:TestPoint
- added TP3: VBUS, TestPoint:TestPoint_Pad_D1.0mm, symbol Connector:TestPoint
- added TP4: PMID, TestPoint:TestPoint_Pad_D1.0mm, symbol Connector:TestPoint
- added TP5: SYS, TestPoint:TestPoint_Pad_D1.0mm, symbol Connector:TestPoint
- added TP6: BAT, TestPoint:TestPoint_Pad_D1.0mm, symbol Connector:TestPoint
- added TP7: GND, TestPoint:TestPoint_Pad_D1.0mm, symbol Connector:TestPoint
- added TP8: 3V3, TestPoint:TestPoint_Pad_D1.0mm, symbol Connector:TestPoint
- added TP9: SCL, TestPoint:TestPoint_Pad_D1.0mm, symbol Connector:TestPoint
- added U7: INA219AIDCNR, Package_TO_SOT_SMD:SOT-23-8, symbol Sensor_Energy:INA219AxDCN
- C16: footprint Capacitor_SMD:C_0603_1608Metric -> Capacitor_SMD:C_0402_1005Metric; LCSC C14663 -> C1525
- C9: value 100n -> 100n/50V; footprint Capacitor_SMD:C_0603_1608Metric -> Capacitor_SMD:C_0402_1005Metric; LCSC C14663 -> C131394
- D1, D2: value SS34 -> SS54; LCSC C8678 -> C22452
- L1: value 2.2uH 3.2A -> 2.2uH 4A molded (MWSA0402S); footprint xiao_solar:IND-SMD_L4.0-W4.0_FNR40XXS -> xiao_solar:IND-SMD_L4.4-W4.2_MWSA0402S; LCSC C167869 -> C408335
- Q2: value AO3400A (ship FET) -> AO3400A
- TP2: value QON (to GND = wake) -> QON
Connections:
- net 3V3: now also TP8.1, U7.4 (VS)
- net BAT: now also JP3.1 (A), TP6.1
- net BATT+: now also RS1.1, U7.1 (IN+); no longer Q2.3 (D), R8.1
- net GND: now also D5.2 (GND), D5.4 (NC), D5.5 (~{ST}), TP7.1, U7.3 (GND), U7.7 (A0), U7.8 (A1)
- net PMID: now also TP4.1
- net SCL: now also TP9.1, U7.5 (SCL)
- net SDA: now also TP10.1, U7.6 (SDA)
- net SYS: now also D5.1 (VIN), TP5.1
- net VBUS: now also TP3.1
- net XIAO_5V: now also D5.3 (~{CE}), D5.6 (VOUT)
- new net BATS: JP3.2 (B), Q2.3 (D), R8.1, RS1.2, TP11.1, U7.2 (IN-)
- no-connect marks 21 -> 8
Other:
- note added: "3V3 идва от регулатора на Xiao."
- note added: "5. I2C (SCL=D6, SDA=D7): BQ25798 0x6B, SHT40 0x44, INA219 0x40"
- note added: "6. Тест точки за първото пускане (падове 1 mm отгоре)"
- note added: "CE: JP2 1-2 (Li-ion) зарежда и без Xiao; 2-3 (LiFePO4) само след запис на VREG и D0=0."
- note added: "D5 (идеален диод LM66100): SYS към пина 5V на Xiao (USB на Xiao не захранва SYS)."
- note added: "DW01A: 2.4 V / 4.3 V резерв, HJ8205 в минуса."
- note added: "PWR_FLAG и отвори"
- note added: "Q2: D към батерията, S към BAT; в shutdown (SDRV_CTRL=01, 0.5 uA)"
- note added: "SS54 = OR на двата входа + защита от обратна полярност. VAC1=VAC2=VBUS, ACDRV към GND (без ACFET)."
- note added: "Watchdog off. D+/D- не се ползват. TP2 (QON) към GND за 1 s = събуждане от ship mode."
- note added: "диодът на Q2 спира разреждането; събужда се, когато панелът даде напрежение."
- note removed: "5. I2C (SCL=D6, SDA=D7): BQ25798 0x6B, SHT40 0x44, PCA9685 0x41"
- note removed: "6. ИЗХОДИ ЗА ТОВАРИ (PWM, до 2 A): нагревател, вентилатор, резерв"
- note removed: "CE: JP2 1-2 (Li-ion) зарежда и без Xiao; 2-3 (LiFePO4) само след запис на VREG и D0=0. Watchdog off. D+/D- не се ползват."
- note removed: "D5: SYS към пина 5V на Xiao (USB на Xiao не захранва SYS). 3V3 идва от регулатора на Xiao."
- note removed: "Q2: D към батерията, S към BAT; в shutdown (SDRV_CTRL=01, 0.5 uA) диодът на Q2 спира разреждането,"
- note removed: "SS34 = OR на двата входа + защита от обратна полярност. VAC1=VAC2=VBUS, ACDRV към GND (без ACFET)."
- note removed: "събужда се само когато се появи напрежение от панела. DW01A: 2.4 V / 4.3 V резерв, HJ8205 в минуса."
